File: LED_driver_DB/LED_driver_DB.kicad_pcb (KiCad board)
At the start: 2 copper layers, 18.4 x 18.4 mm, 6 parts, among them J6 Conn_01x06, U1 STHS34PF80TR

Commit message: change buck converter to TPS563201, production files generated
Parts:
- added G***: LOGO, LOGO, B.Cu at (34.5, 21.2)
