File: LED_driver_MB/LED_driver_MB.kicad_pcb (KiCad board)
At the start: 2 copper layers, 77 x 94.5 mm, 74 parts, among them IC1 MP2393GTL-Z, J1 Conn_01x03_Socket, J2 Conn_01x03_Socket, J3 Conn_01x03_Socket, J4 Conn_01x02_Socket, J5 Conn_01x03_Socket, J6 Conn_01x06, Q1 IRLZ44NPBF, Q10 BC847, Q11 IRLZ44NPBF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

Commit message: change buck converter to TPS563201, production files generated
Parts:
- removed C2: 1u, Capacitor_SMD:C_0603_1608Metric
- removed C3: 10u, Capacitor_SMD:C_1206_3216Metric
- removed C5: 6.8n, Capacitor_SMD:C_0603_1608Metric
- removed D1: LED, LED_SMD:LED_0603_1608Metric
- removed IC1: MP2393GTL-Z, SamacSys_Parts:SOTFL50P160X60-8N
- removed L1: 4.9uH, Inductor_SMD:L_10.4x10.4_H4.8
- removed R1: 20, Resistor_SMD:R_0603_1608Metric
- removed R3: 40.2k, Resistor_SMD:R_0603_1608Metric
- removed R4: 15k, Resistor_SMD:R_0603_1608Metric
- removed R5: 7.68k, Resistor_SMD:R_0603_1608Metric
- added C51: 100nF, Capacitor_SMD:C_0603_1608Metric_Pad1.08x0.95mm_HandSolder, F.Cu at (152.9, 115.3)
- added C52: 100n, Capacitor_SMD:C_0603_1608Metric, F.Cu at (155.6, 108.0)
- added C53: 22u, Capacitor_SMD:C_1206_3216Metric, F.Cu at (145.3, 103.6)
- added C54: 22u, Capacitor_SMD:C_1206_3216Metric, F.Cu at (136.4, 104.1)
- added C81: 22u, Capacitor_SMD:C_1206_3216Metric, F.Cu at (150.7, 111.9)
- added C84: 100nF, Capacitor_SMD:C_0603_1608Metric_Pad1.08x0.95mm_HandSolder, F.Cu at (131.7, 106.2)
- added G***: LOGO, LOGO, F.Cu at (136.9, 95.2)
- added L2: 3.3uH, Inductor_SMD:L_Wuerth_HCM-1350, F.Cu at (141.5, 111.9)
- added R41: 56.2k, Resistor_SMD:R_0603_1608Metric, B.Cu at (159.4, 112.0)
- added R43: 10k, Resistor_SMD:R_0603_1608Metric, B.Cu at (161.0, 112.0)
- added U6: TPS563201, Package_TO_SOT_SMD:SOT-23-6, F.Cu at (155.1, 111.9)
- R2: moved to B.Cu
- moved R2 6.67 mm to (156.7, 118.4)
- moved D2 3.87 mm to (158.4, 105.3), turned to 0 degrees
- moved R24 3.14 mm to (161.8, 107.2)
- moved R25 1.55 mm to (131.7, 107.8)
- moved D3 1.52 mm to (130.0, 110.5)
- moved C4 0.13 mm to (132.6, 111.1)
Connections:
- R2 pad 2: Net-(IC1-EN) -> /5V/EN
- SW1 pad 1: unconnected-(SW1-A-Pad1) -> GND
Routing:
- net /5V/EN: track 0.00 -> 7.65 mm, vias 0 -> 1
- net Net-(IC1-FB): track 5.47 -> 0.00 mm
- net Net-(IC1-SW): track 5.43 -> 0.00 mm
- net Net-(SW1-C): track 17.6 -> 12.4 mm, vias 1 -> 0
- net Net-(U6-SW): track 0.00 -> 5.00 mm, vias 0 -> 7
- net Net-(U6-VFB): track 0.00 -> 4.80 mm, vias 0 -> 1
- net +5V: track 298.4 -> 302.8 mm, vias 31 -> 30
- net Net-(IC1-SS): track 3.23 -> 0.00 mm
- net Net-(IC1-BST): track 3.19 -> 0.00 mm
- net Net-(R3-Pad1): track 3.18 -> 0.00 mm
- net Net-(U6-VBST): track 0.00 -> 3.03 mm
- net Net-(D3-A): track 5.24 -> 2.22 mm
- net Net-(D1-A): track 2.95 -> 0.00 mm
- net Net-(IC1-EN): track 2.66 -> 0.00 mm
- net Net-(C2-Pad1): track 2.21 -> 0.00 mm
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- added copper zone on F.Cu, net Net-(U6-SW)
- removed copper zone on F.Cu, net Net-(IC1-SW)
Other:
- board text added: "Designed by wozniak_works"

Commit message: Via size unified
Routing:
- net Net-(U6-SW): vias 7 -> 5
